File: pixelpad.kicad_sch (KiCad schematic)
At the start: 16 parts, among them SW1 SW_Push_45deg, SW2 SW_Push_45deg, SW3 SW_Push_45deg, SW4 SW_Push_45deg, SW5 SW_Push_45deg, SW6 RotaryEncoder_Switch, U1 MOUDLE-SEEEDUINO-XIAO, U2 ER_OLEDM0.91_1x-I2C

Commit message: Added stuff to the pcb editor
Parts:
- SW1, SW2, SW3, SW4, SW5: footprint (none) -> Button_Switch_Keyboard:SW_Cherry_MX_1.00u_PCB
- SW6: footprint (none) -> Rotary_Encoder:RotaryEncoder_Alps_EC11E-Switch_Vertical_H20mm
Changed lines of the file:
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@@
 			)
 		)
-		(property "Footprint" ""
+		(property "Footprint" "Button_Switch_Keyboard:SW_Cherry_MX_1.00u_PCB"
 			(at 59.69 35.56 0)
 			(hide yes)
@@
 			)
 		)
-		(property "Footprint" ""
+		(property "Footprint" "Button_Switch_Keyboard:SW_Cherry_MX_1.00u_PCB"
 			(at 80.01 59.69 0)
 			(hide yes)
@@
 			)
 		)
-		(property "Footprint" ""
+		(property "Footprint" "Button_Switch_Keyboard:SW_Cherry_MX_1.00u_PCB"
 			(at 39.37 59.69 0)
 			(hide yes)
@@
 			)
 		)
-		(property "Footprint" ""
+		(property "Footprint" "Button_Switch_Keyboard:SW_Cherry_MX_1.00u_PCB"
 			(at 59.69 59.69 0)
 			(hide yes)
@@
 			)
 		)
-		(property "Footprint" ""
+		(property "Footprint" "Rotary_Encoder:RotaryEncoder_Alps_EC11E-Switch_Vertical_H20mm"
 			(at 173.99 73.914 0)
 			(hide yes)
@@
 			)
 		)
-		(property "Footprint" ""
+		(property "Footprint" "Button_Switch_Keyboard:SW_Cherry_MX_1.00u_PCB"
 			(at 39.37 35.56 0)
 			(hide yes)

Commit message: Fully wired up!
Parts:
- renumbered D4 to D3, D5 to D4, D3 to D5, D7 to D6, D6 to D7
Connections:
- net COL0: now also SW3.1; no longer SW4.1
- net COL1: now also SW4.1; no longer SW5.1
- net COL2: now also SW5.1; no longer SW3.1
- net at SW3.2: now also D6.2 (A); no longer D8.2 (A)
- net at SW4.2: now also D7.2 (A); no longer D6.2 (A)
- net at SW5.2: now also D8.2 (A); no longer D7.2 (A)
Other:
- moved on the sheet: SW3, SW4, SW5
Changed lines of the file:
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@@
 	(wire
 		(pts
-			(xy 72.39 57.15) (xy 77.47 57.15)
+			(xy 72.39 27.94) (xy 72.39 33.02)
 		)
 		(stroke
@@
 	(wire
 		(pts
-			(xy 72.39 27.94) (xy 72.39 33.02)
+			(xy 20.32 109.22) (xy 26.67 109.22)
 		)
 		(stroke
@@
 	(wire
 		(pts
-			(xy 20.32 109.22) (xy 26.67 109.22)
+			(xy 60.96 101.6) (xy 60.96 99.06)
 		)
 		(stroke
@@
 	(wire
 		(pts
-			(xy 60.96 101.6) (xy 60.96 99.06)
+			(xy 78.74 33.02) (xy 72.39 33.02)
 		)
 		(stroke
@@
 	(wire
 		(pts
-			(xy 78.74 33.02) (xy 72.39 33.02)
+			(xy 62.23 62.23) (xy 62.23 64.77)
 		)
 		(stroke
@@
 	(wire
 		(pts
+			(xy 52.07 57.15) (xy 57.15 57.15)
+		)
+		(stroke
+			(width 0)
+			(type default)
+		)
+	)
+	(wire
+		(pts
 			(xy 167.64 34.29) (xy 171.45 34.29)
 		)
@@
 	(wire
 		(pts
-			(xy 52.07 57.15) (xy 57.15 57.15)
+			(xy 60.96 116.84) (xy 60.96 118.11)
 		)
 		(stroke
@@
 	(wire
 		(pts
-			(xy 60.96 116.84) (xy 60.96 118.11)
+			(xy 82.55 62.23) (xy 82.55 64.77)
 		)
 		(stroke
@@
 	(wire
 		(pts
+			(xy 31.75 57.15) (xy 36.83 57.15)
+		)
+		(stroke
+			(width 0)
+			(type default)
+		)
+	)
+	(wire
+		(pts
 			(xy 193.04 80.01) (xy 173.99 80.01)
 		)
@@
 	(wire
 		(pts
+			(xy 41.91 62.23) (xy 41.91 64.77)
+		)
+		(stroke
+			(width 0)
+			(type default)
+		)
+	)
+	(wire
+		(pts
 			(xy 34.29 118.11) (xy 34.29 116.84)
 		)
@@
 	(wire
 		(pts
-			(xy 167.64 26.67) (xy 185.42 26.67)
+			(xy 72.39 57.15) (xy 77.47 57.15)
 		)
 		(stroke
@@
 	(wire
 		(pts
-			(xy 82.55 64.77) (xy 82.55 62.23)
+			(xy 167.64 26.67) (xy 185.42 26.67)
 		)
 		(stroke
@@
 	(wire
 		(pts
-			(xy 41.91 64.77) (xy 41.91 62.23)
-		)
-		(stroke
-			(width 0)
-			(type default)
-		)
-	)
-	(wire
-		(pts
 			(xy 124.6489 78.7399) (xy 124.6489 83.8199)
 		)
@@
 	(wire
 		(pts
-			(xy 62.23 64.77) (xy 62.23 62.23)
-		)
-		(stroke
-			(width 0)
-			(type default)
-		)
-	)
-	(wire
-		(pts
 			(xy 78.74 33.02) (xy 78.74 35.56)
 		)
@@
 	(wire
 		(pts
-			(xy 31.75 57.15) (xy 36.83 57.15)
-		)
-		(stroke
-			(width 0)
-			(type default)
-		)
-	)
-	(wire
-		(pts
 			(xy 34.29 99.06) (xy 34.29 101.6)
 		)
@@
 	(symbol
 		(lib_id "KiCad-User:SW_Push_45deg")
-		(at 80.01 59.69 0)
+		(at 39.37 59.69 0)
 		(unit 1)
 		(body_style 1)
@@
 		(fields_autoplaced yes)
 		(property "Reference" "SW3"
-			(at 80.01 52.07 0)
+			(at 39.37 52.07 0)
 			(show_name no)
 			(do_not_autoplace no)
@@
 		)
 		(property "Value" "SW_Push_45deg"
-			(at 80.01 54.61 0)
+			(at 39.37 54.61 0)
 			(show_name no)
 			(do_not_autoplace no)
@@
 		)
 		(property "Footprint" "Button_Switch_Keyboard:SW_Cherry_MX_1.00u_PCB"
-			(at 80.01 59.69 0)
+			(at 39.37 59.69 0)
 			(hide yes)
 			(show_name no)
@@
 		)
 		(property "Datasheet" ""
-			(at 80.01 59.69 0)
+			(at 39.37 59.69 0)
 			(hide yes)
 			(show_name no)
@@
 		)
 		(property "Description" "Push button switch, normally open, two pins, 45° tilted"
-			(at 80.01 59.69 0)
+			(at 39.37 59.69 0)
 			(hide yes)
 			(show_name no)
@@
 	(symbol
 		(lib_id "KiCad-User:SW_Push_45deg")
-		(at 39.37 59.69 0)
+		(at 59.69 59.69 0)
 		(unit 1)
 		(body_style 1)
@@
 		(fields_autoplaced yes)
 		(property "Reference" "SW4"
-			(at 39.37 52.07 0)
+			(at 59.69 52.07 0)
 			(show_name no)
 			(do_not_autoplace no)
@@
 		)
 		(property "Value" "SW_Push_45deg"
-			(at 39.37 54.61 0)
+			(at 59.69 54.61 0)
 			(show_name no)
 			(do_not_autoplace no)
@@
 		)
 		(property "Footprint" "Button_Switch_Keyboard:SW_Cherry_MX_1.00u_PCB"
-			(at 39.37 59.69 0)
+			(at 59.69 59.69 0)
 			(hide yes)
 			(show_name no)
@@
 		)
 		(property "Datasheet" ""
-			(at 39.37 59.69 0)
+			(at 59.69 59.69 0)
 			(hide yes)
 			(show_name no)
@@
 		)
 		(property "Description" "Push button switch, normally open, two pins, 45° tilted"
-			(at 39.37 59.69 0)
+			(at 59.69 59.69 0)
 			(hide yes)
 			(show_name no)
@@
 		(dnp no)
 		(fields_autoplaced yes)
-		(property "Reference" "D7"
+		(property "Reference" "D6"
 			(at 44.45 67.3099 90)
 			(show_name no)
@@
 			(project "pixelpad"
 				(path "/3414973a-652a-4c78-88cc-120293b3a4e8"
-					(reference "D7")
+					(reference "D6")
 					(unit 1)
 				)
@@
 		(dnp no)
 		(fields_autoplaced yes)
-		(property "Reference" "D3"
+		(property "Reference" "D5"
 			(at 88.9 43.1799 90)
 			(show_name no)
@@
 			(project "pixelpad"
 				(path "/3414973a-652a-4c78-88cc-120293b3a4e8"
-					(reference "D3")
+					(reference "D5")
 					(unit 1)
 				)
@@
 		(dnp no)
 		(fields_autoplaced yes)
-		(property "Reference" "D4"
+		(property "Reference" "D3"
 			(at 44.45 43.1799 90)
 			(show_name no)
@@
 			(project "pixelpad"
 				(path "/3414973a-652a-4c78-88cc-120293b3a4e8"
-					(reference "D4")
+					(reference "D3")
 					(unit 1)
 				)
@@
 		(dnp no)
 		(fields_autoplaced yes)
-		(property "Reference" "D5"
+		(property "Reference" "D4"
 			(at 64.77 43.1799 90)
 			(show_name no)
@@
 			(project "pixelpad"
 				(path "/3414973a-652a-4c78-88cc-120293b3a4e8"
-					(reference "D5")
+					(reference "D4")
 					(unit 1)
 				)
@@
 	(symbol
 		(lib_id "KiCad-User:SW_Push_45deg")
-		(at 59.69 59.69 0)
+		(at 80.01 59.69 0)
 		(unit 1)
 		(body_style 1)
@@
 		(fields_autoplaced yes)
 		(property "Reference" "SW5"
-			(at 59.69 52.07 0)
+			(at 80.01 52.07 0)
 			(show_name no)
 			(do_not_autoplace no)
@@
 		)
 		(property "Value" "SW_Push_45deg"
-			(at 59.69 54.61 0)
+			(at 80.01 54.61 0)
 			(show_name no)
 			(do_not_autoplace no)
@@
 		)
 		(property "Footprint" "Button_Switch_Keyboard:SW_Cherry_MX_1.00u_PCB"
-			(at 59.69 59.69 0)
+			(at 80.01 59.69 0)
 			(hide yes)
 			(show_name no)
@@
 		)
 		(property "Datasheet" ""
-			(at 59.69 59.69 0)
+			(at 80.01 59.69 0)
 			(hide yes)
 			(show_name no)
@@
 		)
 		(property "Description" "Push button switch, normally open, two pins, 45° tilted"
-			(at 59.69 59.69 0)
+			(at 80.01 59.69 0)
 			(hide yes)
 			(show_name no)
@@
 		(dnp no)
 		(fields_autoplaced yes)
-		(property "Reference" "D6"
+		(property "Reference" "D7"
 			(at 64.77 67.3099 90)
 			(show_name no)
@@
 			(project "pixelpad"
 				(path "/3414973a-652a-4c78-88cc-120293b3a4e8"
-					(reference "D6")
+					(reference "D7")
 					(unit 1)
 				)
