File: pcb/pixelpad.kicad_pcb (KiCad board)
At the start: 2 copper layers, 61.5 x 55.5 mm, 18 parts, among them J1 OLED Display, SW1 SW_Push_45deg, SW2 SW_Push_45deg, SW3 RotaryEncoder_Switch, SW4 SW_Push_45deg, SW5 SW_Push_45deg, SW6 SW_Push_45deg, U1 MOUDLE-SEEEDUINO-XIAO

Commit message: Found out you can put 3d models into kicad 0.0
Parts:
- D1, D2: value WS2812B -> SK6812MINI-E
- J1: footprint Connector_PinHeader_2.54mm:PinHeader_1x04_P2.54mm_Vertical -> XIAO:PinHeader_1x04_P2.54mm_Vertical
- SW1, SW2, SW4, SW5, SW6: footprint Button_Switch_Keyboard:SW_Cherry_MX_1.00u_PCB -> XIAO:SW_Cherry_MX_1.00u_PCB
- moved D2 0.15 mm to (112.0, 45.5)
- turned D1 to 0 degrees
