File: pcb/pixelpad.kicad_sch (KiCad schematic)
At the start: 16 parts, among them J1 OLED Display, SW1 SW_Push_45deg, SW2 SW_Push_45deg, SW3 RotaryEncoder_Switch, SW4 SW_Push_45deg, SW5 SW_Push_45deg, SW6 SW_Push_45deg, U1 MOUDLE-SEEEDUINO-XIAO

Commit message: Found out you can put 3d models into kicad 0.0
Parts:
- D1, D2: footprint SK6812MINI-E - 3.2x2.8x1.78mm -> XIAO:SK6812MINI-E_fixed
- J1: footprint Connector_PinHeader_2.54mm:PinHeader_1x04_P2.54mm_Vertical -> XIAO:PinHeader_1x04_P2.54mm_Vertical
- SW1, SW2, SW4, SW5, SW6: footprint Button_Switch_Keyboard:SW_Cherry_MX_1.00u_PCB -> XIAO:SW_Cherry_MX_1.00u_PCB
Changed lines of the file:
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@@
 			)
 		)
-		(property "Footprint" "Connector_PinHeader_2.54mm:PinHeader_1x04_P2.54mm_Vertical"
+		(property "Footprint" "XIAO:PinHeader_1x04_P2.54mm_Vertical"
 			(at 124.46 66.04 0)
 			(hide yes)
@@
 			)
 		)
-		(property "Footprint" "Button_Switch_Keyboard:SW_Cherry_MX_1.00u_PCB"
+		(property "Footprint" "XIAO:SW_Cherry_MX_1.00u_PCB"
 			(at 59.69 35.56 0)
 			(hide yes)
@@
 			)
 		)
-		(property "Footprint" "SK6812MINI-E - 3.2x2.8x1.78mm"
+		(property "Footprint" "XIAO:SK6812MINI-E_fixed"
 			(at 39.37 119.38 0)
 			(hide yes)
@@
 			)
 		)
-		(property "Footprint" "Button_Switch_Keyboard:SW_Cherry_MX_1.00u_PCB"
+		(property "Footprint" "XIAO:SW_Cherry_MX_1.00u_PCB"
 			(at 39.37 62.23 0)
 			(hide yes)
@@
 			)
 		)
-		(property "Footprint" "Button_Switch_Keyboard:SW_Cherry_MX_1.00u_PCB"
+		(property "Footprint" "XIAO:SW_Cherry_MX_1.00u_PCB"
 			(at 59.69 62.23 0)
 			(hide yes)
@@
 			)
 		)
-		(property "Footprint" "SK6812MINI-E - 3.2x2.8x1.78mm"
+		(property "Footprint" "XIAO:SK6812MINI-E_fixed"
 			(at 66.04 119.38 0)
 			(hide yes)
@@
 			)
 		)
-		(property "Footprint" "Button_Switch_Keyboard:SW_Cherry_MX_1.00u_PCB"
+		(property "Footprint" "XIAO:SW_Cherry_MX_1.00u_PCB"
 			(at 39.37 35.56 0)
 			(hide yes)
@@
 			)
 		)
-		(property "Footprint" "Button_Switch_Keyboard:SW_Cherry_MX_1.00u_PCB"
+		(property "Footprint" "XIAO:SW_Cherry_MX_1.00u_PCB"
 			(at 80.01 62.23 0)
 			(hide yes)
